File: pcb/CBB.kicad_pcb (KiCad board)
At the start: 2 copper layers, 43.8 x 31.8 mm, 33 parts, among them J1 Conn_01x03_Pin, J2 Conn_01x04_Pin, J3 Conn_01x05_Pin, J4 Conn_01x02_Pin, J5 Conn_01x02_Pin, J6 Conn_01x03_Pin, J7 Conn_01x03_Pin, J8 Conn_01x02_Pin, J9 Screw_Terminal_01x03, U1 MCP2518FD-xSL, U2 ATtiny1606-S, U3 ATA6563-GAQW1, Y1 4MHz

Commit message: Update to KiCAD 9
Parts:
- moved Y1 0.13 mm to (141.2, 82.8)
