File: pcb/CBB.kicad_sch (KiCad schematic)
At the start: 33 parts, among them J1 Conn_01x03_Pin, J2 Conn_01x04_Pin, J3 Conn_01x05_Pin, J4 Conn_01x02_Pin, J5 Conn_01x02_Pin, J6 Conn_01x03_Pin, J7 Conn_01x03_Pin, J8 Conn_01x02_Pin, J9 Screw_Terminal_01x03, U1 MCP2518FD-xSL, U2 ATtiny1606-S, U3 ATA6563-GAQW1, Y1 4MHz

Commit message: Update to KiCAD 9
Parts:
- FID1, FID2, FID3, FID4, JP1, JP2: now left out of the parts list

Commit message: Rename/Add/Remove bom fields
Parts:
- C1, C5: HTL (none) -> 103620; Vendor HTL -> (none); VendorId 103620 -> (none)
- C2, C3, C4, C6: HTL (none) -> 100128; Vendor HTL -> (none); VendorId 100128 -> (none)
- C7, C8: HTL (none) -> 100105; Vendor HTL -> (none); VendorId 100105 -> (none)
- J1, J2, J3, J4, J5, J6, J7, J8: HTL (none) -> 101521; Vendor HTL -> (none); VendorId 101521 -> (none)
- J9: DigiKey (none) -> 277-1107-ND, 277-1012-ND; Vendor DigiKey -> (none); VendorId 277-1107-ND, 277-1012-ND -> (none)
- R1, R2, R3, R4: HTL (none) -> 102951; Vendor HTL -> (none); VendorId 102951 -> (none)
- R5: HTL (none) -> 102933; Vendor HTL -> (none); VendorId 102933 -> (none)
- U1: DigiKey (none) -> MCP2518FDT-E/SLCT-ND; Vendor HTL -> (none); VendorId MCP2518FDT-E/SLCT-ND -> (none)
- U2: HTL (none) -> 103450; Vendor HTL -> (none); VendorId 103450 -> (none)
- U3: DigiKey (none) -> 150-ATA6563-GAQW1CT-ND; Vendor DigiKey -> (none); VendorId 150-ATA6563-GAQW1CT-ND -> (none)
- Y1: DigiKey (none) -> 1908-J49SMH-A-G-G-K-4M0CT-ND; Vendor DigiKey -> (none); VendorId 1908-J49SMH-A-G-G-K-4M0CT-ND -> (none)
